File: hw/step_load.kicad_pcb (KiCad board)
At the start: 4 copper layers, 160 x 100 mm, 186 parts, among them J1 DC_IN, J2 USB_C_Receptacle_USB2.0_16P, J3 OUTPUT, J4 OLED, J5 UART, J6 BOOT, K1 G6K-2F-Y, K10 G6K-2F-Y, K11 G6K-2F-Y, K12 G6K-2F-Y, K13 G6K-2F-Y, K14 G6K-2F-Y, K15 G6K-2F-Y, K16 G6K-2F-Y, K2 G6K-2F-Y, K3 G6K-2F-Y, K4 G6K-2F-Y, K5 G6K-2F-Y, K6 G6K-2F-Y, K7 G6K-2F-Y, K8 G6K-2F-Y, K9 G6K-2F-Y, Q1 Si2302CDS, Q10 Si2302CDS, Q11 Si2302CDS, Q12 Si2302CDS, Q13 Si2302CDS, Q14 Si2302CDS, Q15 Si2302CDS, Q16 Si2302CDS, Q2 Si2302CDS, Q3 Si2302CDS, Q4 Si2302CDS, Q5 Si2302CDS, Q6 Si2302CDS, Q7 Si2302CDS, Q8 Si2302CDS, Q9 Si2302CDS, SW1 RST, SW2 RST, SW3 RST, SW4 RST, U1 AZ1117-3.3, U2 TCA9535PWR, U3 LM35DZ, U4 LM35DZ, U5 ESP32-C3-WROOM-02

Commit message: pcb update
Parts:
- moved D11 168.5 mm to (-37.8, -6.25)
- moved D13 168.2 mm to (-33.8, -6.25)
- moved C24 167.9 mm to (-42.2, -0.06)
- moved Q4 167.1 mm to (-42.2, -3.06), turned to 90 degrees
- moved R20 164.9 mm to (-43.8, -5.56), turned to 90 degrees
- moved R18 163.0 mm to (-42.2, 1.69), turned to 180 degrees
- moved K4 161.5 mm to (-35.0, 0.00)
- moved D10 133.1 mm to (-52.8, -6.25)
- moved R19 130.5 mm to (-58.5, -5.50), turned to 90 degrees
- moved C23 129.8 mm to (-57.0, 0.00)
- moved D12 127.4 mm to (-48.8, -6.25)
- moved Q3 123.4 mm to (-57.0, -2.94), turned to 90 degrees
- moved C4 122.1 mm to (54.1, 94.1)
- moved R1 122.1 mm to (46.1, 91.1)
- moved U2 122.1 mm to (49.1, 97.1)
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
Commit message: pcb update
Parts:
- moved C28 246.9 mm to (186.0, 78.2)
- moved Q8 246.9 mm to (186.0, 75.2)
- moved R30 246.9 mm to (186.0, 80.0)
- moved R32 246.9 mm to (184.5, 72.8)
- moved C32 246.4 mm to (186.0, 101.8)
- moved Q12 246.4 mm to (186.0, 98.8)
- moved R42 246.4 mm to (186.0, 103.5)
- moved R44 246.4 mm to (184.5, 96.2)
- moved C36 246.2 mm to (185.9, 126.0)
- moved Q16 246.2 mm to (185.9, 123.0)
- moved R54 246.2 mm to (185.9, 127.8)
- moved R56 246.2 mm to (184.4, 120.5)
- moved D19 245.9 mm to (189.8, 72.0)
- moved D21 245.9 mm to (193.8, 72.0)
- moved K8 245.9 mm to (192.5, 78.2)
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
Commit message: pcb update
Parts:
- added J7: DC_IN, Connector_PinHeader_2.54mm:PinHeader_1x02_P2.54mm_Vertical, F.Cu at (122.0, 54.0)
- moved R4 159.3 mm to (106.0, 45.0), turned to 90 degrees
- moved D3 155.8 mm to (106.0, 42.0), turned to 90 degrees
- moved C20 101.6 mm to (92.2, 114.8)
- moved R12 101.6 mm to (98.0, 114.8)
- moved SW4 101.6 mm to (91.8, 106.8)
- moved R5 98.3 mm to (102.0, 137.2), turned to 90 degrees
- moved R11 94.3 mm to (101.5, 106.0), turned to -90 degrees
- moved C19 93.6 mm to (104.5, 105.0), turned to 0 degrees
- moved R9 91.8 mm to (97.8, 101.0)
- moved D4 91.6 mm to (102.0, 134.2), turned to 90 degrees
- moved J6 90.8 mm to (107.0, 99.5), turned to 180 degrees
- moved C14 89.7 mm to (93.0, 103.0)
- moved R6 87.3 mm to (114.5, 134.2), turned to 90 degrees
- moved SW1 87.0 mm to (105.5, 133.8)
- moved R1 86.0 mm to (132.0, 87.1), turned to -90 degrees
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Routing:
- net USB_ESP+: track 0.00 -> 2.78 mm
- net USB_ESP-: track 0.00 -> 2.78 mm

Commit message: pcb update
Parts:
- moved R11 12.2 mm to (111.2, 98.8), turned to 90 degrees
- moved C20 11.0 mm to (101.2, 108.5)
- moved C19 8.19 mm to (109.8, 98.8), turned to 90 degrees
- moved R12 5.77 mm to (101.2, 110.0)
- moved C4 4.00 mm to (128.0, 92.0)
- moved R1 4.00 mm to (128.0, 87.1)
- moved U2 4.00 mm to (123.0, 90.0)
- moved R7 2.49 mm to (95.8, 102.3), turned to 90 degrees
- moved C15 1.95 mm to (91.5, 102.2), turned to -90 degrees
- moved SW4 1.75 mm to (91.8, 108.5)
- moved R9 1.44 mm to (97.2, 102.3), turned to 90 degrees
- moved C14 0.78 mm to (93.0, 102.2), turned to -90 degrees
- moved U5 0.25 mm to (97.5, 90.0)
- moved Q5 0.06 mm to (141.0, 75.2)
Routing:
- net GND: vias 0 -> 7

Commit message: sch & pcb update
Parts:
- added D38: B3V6, Diode_SMD:D_SOD-523, F.Cu at (132.8, 50.0)
- added R61: 10, Resistor_SMD:R_0603_1608Metric, F.Cu at (141.0, 57.2)
- added R62: 10, Resistor_SMD:R_0603_1608Metric, F.Cu at (156.0, 57.2)
- added R63: 10, Resistor_SMD:R_0603_1608Metric, F.Cu at (171.0, 57.2)
- added R64: 10, Resistor_SMD:R_0603_1608Metric, F.Cu at (186.0, 57.2)
- added R65: 10, Resistor_SMD:R_0603_1608Metric, F.Cu at (140.9, 81.5)
- added R66: 10, Resistor_SMD:R_0603_1608Metric, F.Cu at (156.0, 81.5)
- added R67: 10, Resistor_SMD:R_0603_1608Metric, F.Cu at (171.0, 81.5)
- added R68: 10, Resistor_SMD:R_0603_1608Metric, F.Cu at (186.0, 81.5)
- added R69: 10, Resistor_SMD:R_0603_1608Metric, F.Cu at (141.0, 105.5)
- added R70: 10, Resistor_SMD:R_0603_1608Metric, F.Cu at (156.0, 105.2)
- added R71: 10, Resistor_SMD:R_0603_1608Metric, F.Cu at (171.0, 105.2)
- added R72: 10, Resistor_SMD:R_0603_1608Metric, F.Cu at (186.0, 105.0)
- added R73: 10, Resistor_SMD:R_0603_1608Metric, F.Cu at (141.0, 129.2)
- added R74: 10, Resistor_SMD:R_0603_1608Metric, F.Cu at (156.0, 129.2)
- added R75: 10, Resistor_SMD:R_0603_1608Metric, F.Cu at (171.0, 129.2)
- added R76: 10, Resistor_SMD:R_0603_1608Metric, F.Cu at (185.8, 129.2)
- added R77: 10, Resistor_SMD:R_0603_1608Metric, F.Cu at (129.8, 50.0)
- added R78: 10, Resistor_SMD:R_0603_1608Metric, F.Cu at (131.2, 50.0)
- moved C5 8.13 mm to (116.3, 78.8), turned to 0 degrees
- moved C2 5.30 mm to (116.3, 76.8), turned to 0 degrees
- moved C4 4.50 mm to (132.5, 92.0)
- moved R1 4.50 mm to (132.5, 87.1)
- moved U2 4.50 mm to (127.5, 90.0)
- moved D5 3.75 mm to (128.0, 49.8)
- moved NT1 0.50 mm to (130.5, 45.0)
- moved NT2 0.50 mm to (133.0, 45.0)
- moved J7 0.25 mm to (122.0, 54.2)
- moved C6 0.25 mm to (119.8, 60.0)
- moved J5 0.12 mm to (135.5, 42.0)
Connections:
- C21 pad 1: /P00 -> Net-(Q1-G)
- C22 pad 1: /P04 -> Net-(Q2-G)
- C23 pad 1: /P10 -> Net-(Q3-G)
- C24 pad 1: /P14 -> Net-(Q4-G)
- C25 pad 1: /P01 -> Net-(Q5-G)
- C26 pad 1: /P05 -> Net-(Q6-G)
- C27 pad 1: /P11 -> Net-(Q7-G)
- C28 pad 1: /P15 -> Net-(Q8-G)
- C29 pad 1: /P02 -> Net-(Q9-G)
- C30 pad 1: /P06 -> Net-(Q10-G)
- C31 pad 1: /P12 -> Net-(Q11-G)
- C32 pad 1: /P16 -> Net-(Q12-G)
- C33 pad 1: /P03 -> Net-(Q13-G)
- C34 pad 1: /P07 -> Net-(Q14-G)
- C35 pad 1: /P13 -> Net-(Q15-G)
- C36 pad 1: /P17 -> Net-(Q16-G)
- D5 pad 1: +3.3V -> Net-(D5-K)
- Q1 pad 1: /P00 -> Net-(Q1-G)
- Q10 pad 1: /P06 -> Net-(Q10-G)
- Q11 pad 1: /P12 -> Net-(Q11-G)
- Q12 pad 1: /P16 -> Net-(Q12-G)
- Q13 pad 1: /P03 -> Net-(Q13-G)
- Q14 pad 1: /P07 -> Net-(Q14-G)
- Q15 pad 1: /P13 -> Net-(Q15-G)
- Q16 pad 1: /P17 -> Net-(Q16-G)
- Q2 pad 1: /P04 -> Net-(Q2-G)
- Q3 pad 1: /P10 -> Net-(Q3-G)
- Q4 pad 1: /P14 -> Net-(Q4-G)
- Q5 pad 1: /P01 -> Net-(Q5-G)
- Q6 pad 1: /P05 -> Net-(Q6-G)
- Q7 pad 1: /P11 -> Net-(Q7-G)
- Q8 pad 1: /P15 -> Net-(Q8-G)
- Q9 pad 1: /P02 -> Net-(Q9-G)
- R13 pad 2: /P00 -> Net-(Q1-G)
- R14 pad 2: /P04 -> Net-(Q2-G)
- R17 pad 2: /P10 -> Net-(Q3-G)
- R18 pad 2: /P14 -> Net-(Q4-G)
- R25 pad 2: /P01 -> Net-(Q5-G)
- R26 pad 2: /P05 -> Net-(Q6-G)
- R29 pad 2: /P11 -> Net-(Q7-G)
- R30 pad 2: /P15 -> Net-(Q8-G)
- R37 pad 2: /P02 -> Net-(Q9-G)
- R38 pad 2: /P06 -> Net-(Q10-G)
- R41 pad 2: /P12 -> Net-(Q11-G)
- R42 pad 2: /P16 -> Net-(Q12-G)
- R49 pad 2: /P03 -> Net-(Q13-G)
- R50 pad 2: /P07 -> Net-(Q14-G)
- R53 pad 2: /P13 -> Net-(Q15-G)
- R54 pad 2: /P17 -> Net-(Q16-G)
Routing:
- net I2C_SDA: track 0.00 -> 53.6 mm, vias 0 -> 2
- net I2C_SCL: track 0.00 -> 48.2 mm
- net EN: track 0.00 -> 16.8 mm
- net +3.3V: track 0.00 -> 5.28 mm, vias 0 -> 2
- net GND: track 0.00 -> 3.54 mm, vias 7 -> 18
- net /~{INT}: track 0.00 -> 1.77 mm
Other:
- outline, holes or cut-outs redrawn

Commit message: pcb update
Parts:
- moved R7 13.9 mm to (106.5, 93.5), turned to 180 degrees
- moved R9 10.9 mm to (106.5, 96.5), turned to 180 degrees
- moved R11 5.84 mm to (105.5, 99.8), turned to -90 degrees
- moved C19 2.93 mm to (107.0, 99.8), turned to -90 degrees
- moved J6 2.52 mm to (109.5, 99.2), turned to 0 degrees
- moved U5 0.20 mm to (97.3, 90.0)
Routing:
- net USER_BTN3: track 0.00 -> 60.1 mm
- net USER_BTN2: track 0.00 -> 56.1 mm
- net USER_BTN1: track 0.00 -> 51.8 mm
- net GND: track 3.54 -> 45.5 mm, vias 18 -> 52
- net BOOT: track 0.00 -> 9.96 mm
- net I2C_SDA: track 53.6 -> 56.4 mm
- net I2C_SCL: track 48.2 -> 49.6 mm
- net Net-(D4-K): track 0.00 -> 1.39 mm

Commit message: pcb update
Parts:
- moved D27 90.3 mm to (147.5, 132.5)
- moved D23 89.8 mm to (150.8, 134.2), turned to 180 degrees
- moved R55 86.0 mm to (151.0, 132.5), turned to 0 degrees
- moved Q9 80.0 mm to (153.9, 129.2), turned to -90 degrees
- moved K9 78.2 mm to (147.5, 126.2), turned to 180 degrees
- moved D35 76.4 mm to (147.5, 108.5)
- moved D18 75.2 mm to (144.0, 46.2)
- moved R9 74.6 mm to (207.0, 136.2)
- moved C29 74.2 mm to (154.0, 126.2), turned to 180 degrees
- moved D31 73.7 mm to (150.8, 110.2), turned to 180 degrees
- moved D22 73.6 mm to (147.5, 48.0), turned to 180 degrees
- moved C28 73.3 mm to (141.0, 54.2)
- moved K8 73.3 mm to (147.5, 54.2)
- moved Q8 73.3 mm to (141.0, 51.2)
- moved R50 73.3 mm to (141.0, 57.5)
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- renumbered C7 to C1, C20 to C10, C14 to C11, C15 to C12, C1 to C13, C2 to C14, C5 to C15, C8 to C16, C9 to C17, C3 to C18, C6 to C19, C10 to C2, C4 to C20, C25 to C22, C29 to C23, C33 to C24, C22 to C25, C30 to C27, C34 to C28, C23 to C29, C11 to C3, C27 to C30, C35 to C32, C24 to C33, C28 to C34, C32 to C35, C12 to C4, C13 to C5, C16 to C6, C17 to C7, C18 to C8, C19 to C9, D3 to D1, D30 to D10, D8 to D11, D16 to D12, D24 to D13, D32 to D14, D7 to D15, D15 to D16, D23 to D17, D31 to D18, D9 to D19, D4 to D2, D17 to D20, D25 to D21, D33 to D22, D10 to D23, D18 to D24, D26 to D25, D34 to D26, D12 to D27, D20 to D28, D28 to D29, D5 to D3, D36 to D30, D11 to D31, D19 to D32, D27 to D33, D35 to D34, D13 to D35, D21 to D36, D29 to D37, D37 to D38, D38 to D4, D1 to D5, D2 to D6, D6 to D7, D14 to D8, D22 to D9, H3 to H2, H2 to H3, J6 to J1, J5 to J3, J1 to J4, J7 to J5, J4 to J6, J3 to J7, K7 to K10, K15 to K12, K4 to K13, K8 to K14, K12 to K15, K5 to K2, K9 to K3, K13 to K4, K2 to K5, K10 to K7, K14 to K8, K3 to K9, Q7 to Q10, Q15 to Q12, Q4 to Q13, Q8 to Q14, Q12 to Q15, Q5 to Q2, Q9 to Q3, Q13 to Q4, Q2 to Q5, Q10 to Q7, Q14 to Q8, Q3 to Q9, R21 to R1, R35 to R10, R47 to R11, R59 to R12, R24 to R13, R36 to R14, R48 to R15, R60 to R16, R6 to R17, R8 to R18, R10 to R19, R33 to R2, R11 to R20, R12 to R21, R2 to R22, R3 to R23, R4 to R24, R5 to R25, R78 to R26, R77 to R27, R7 to R28, R9 to R29, R45 to R3, R1 to R30, R15 to R31, R27 to R32, R39 to R33, R51 to R34, R61 to R35, R65 to R36, R69 to R37, R73 to R38, R13 to R39, R57 to R4, R25 to R40, R37 to R41, R49 to R42, R16 to R43, R28 to R44, R40 to R45, R52 to R46, R62 to R47, R66 to R48, R70 to R49, R22 to R5, R74 to R50, R14 to R51, R26 to R52, R38 to R53, R50 to R54, R19 to R55, R31 to R56, R43 to R57, R55 to R58, R63 to R59, R34 to R6, R67 to R60, R71 to R61, R75 to R62, R17 to R63, R29 to R64, R41 to R65, R53 to R66, R20 to R67, R32 to R68, R44 to R69, R46 to R7, R56 to R70, R64 to R71, R68 to R72, R72 to R73, R76 to R74, R18 to R75, R30 to R76, R42 to R77, R54 to R78, R58 to R8, R23 to R9, U3 to U1, U4 to U2, U1 to U3, U5 to U4, U2 to U5
Routing:
- net /VNEG: track 0.00 -> 701.9 mm
- net /VPOS: track 0.00 -> 120.2 mm
- net /P13: track 0.00 -> 88.2 mm, vias 0 -> 2
- net /P04: track 0.00 -> 80.4 mm, vias 0 -> 2
- net /P17: track 0.00 -> 75.5 mm, vias 0 -> 2
- net /P12: track 0.00 -> 73.8 mm, vias 0 -> 2
- net /P05: track 0.00 -> 66.4 mm, vias 0 -> 2
- net /P00: track 0.00 -> 62.2 mm, vias 0 -> 2
- net /P16: track 0.00 -> 61.1 mm, vias 0 -> 2
- net /P11: track 0.00 -> 59.5 mm, vias 0 -> 2
- net /P06: track 0.00 -> 52.0 mm, vias 0 -> 2
- net /P01: track 0.00 -> 47.6 mm, vias 0 -> 2
- net /P15: track 0.00 -> 46.0 mm, vias 0 -> 2
- net /P10: track 0.00 -> 45.7 mm, vias 0 -> 2
- net /P07: track 0.00 -> 36.8 mm, vias 0 -> 2
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