File: hw/step_load.kicad_pcb (KiCad board)
At the start: 4 copper layers, 160 x 100 mm, 206 parts, among them J1 BOOT, J2 USB_C_Receptacle_USB2.0_16P, J3 UART, J4 DC_IN, J5 DC_IN, J6 OLED, J7 OUTPUT, K1 G6K-2F-Y, K10 G6K-2F-Y, K11 G6K-2F-Y, K12 G6K-2F-Y, K13 G6K-2F-Y, K14 G6K-2F-Y, K15 G6K-2F-Y, K16 G6K-2F-Y, K2 G6K-2F-Y, K3 G6K-2F-Y, K4 G6K-2F-Y, K5 G6K-2F-Y, K6 G6K-2F-Y, K7 G6K-2F-Y, K8 G6K-2F-Y, K9 G6K-2F-Y, Q1 Si2302CDS, Q10 Si2302CDS, Q11 Si2302CDS, Q12 Si2302CDS, Q13 Si2302CDS, Q14 Si2302CDS, Q15 Si2302CDS, Q16 Si2302CDS, Q2 Si2302CDS, Q3 Si2302CDS, Q4 Si2302CDS, Q5 Si2302CDS, Q6 Si2302CDS, Q7 Si2302CDS, Q8 Si2302CDS, Q9 Si2302CDS, SW1 RST, SW2 RST, SW3 RST, SW4 RST, U1 LM35DZ, U2 LM35DZ, U3 AZ1117-3.3, U4 ESP32-C3-WROOM-02, U5 TCA9535PWR

Commit message: pcb update
Routing:
- net Net-(K12-Pad3): track 10.0 -> 102.0 mm
- net Net-(K9-Pad3): track 10.0 -> 78.5 mm
- net Net-(K13-Pad3): track 10.0 -> 78.2 mm
- net Net-(K5-Pad3): track 10.0 -> 77.2 mm
- net Net-(K10-Pad3): track 10.0 -> 74.2 mm
- net Net-(K14-Pad3): track 10.0 -> 73.0 mm
- net Net-(K11-Pad3): track 10.0 -> 69.2 mm
- net Net-(K15-Pad3): track 10.0 -> 68.1 mm
- net Net-(K16-Pad3): track 10.0 -> 61.7 mm
- net GND: track 62.7 -> 66.0 mm, vias 58 -> 56

Commit message: pcb update
Parts:
- moved R5 21.3 mm to (237.0, 43.0), turned to -90 degrees
- moved R6 21.2 mm to (227.0, 43.0), turned to -90 degrees
- moved R7 21.2 mm to (217.0, 43.0), turned to -90 degrees
- moved R8 21.2 mm to (207.0, 43.0), turned to -90 degrees
- moved R1 20.1 mm to (237.0, 68.2), turned to -90 degrees
- moved R2 19.9 mm to (227.0, 68.2), turned to -90 degrees
- moved R3 19.9 mm to (217.0, 68.2), turned to -90 degrees
- moved R4 19.9 mm to (207.0, 68.2), turned to -90 degrees
- moved C5 9.15 mm to (199.2, 57.5), turned to 180 degrees
- moved D5 1.25 mm to (110.8, 61.3)
- moved D6 1.25 mm to (112.8, 61.3)
- moved R10 0.84 mm to (217.0, 137.0)
- moved R11 0.84 mm to (227.0, 137.0)
- moved R9 0.84 mm to (207.0, 137.0)
- moved R12 0.68 mm to (237.0, 137.0)
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Routing:
- net /VNEG: track 701.9 -> 514.3 mm
- net GND: track 66.0 -> 235.7 mm, vias 56 -> 258
- net TEMP_RES: track 0.00 -> 126.6 mm, vias 0 -> 1
- net /VPOS: track 120.2 -> 242.5 mm
- net Net-(K4-Pad3): track 10.0 -> 77.8 mm
- net Net-(K8-Pad3): track 10.0 -> 74.6 mm
- net Net-(K3-Pad3): track 10.0 -> 73.5 mm
- net Net-(K7-Pad3): track 10.0 -> 71.3 mm
- net Net-(K6-Pad3): track 10.0 -> 68.9 mm
- net ESP_TX: track 0.00 -> 58.4 mm, vias 0 -> 2
- net Net-(K2-Pad3): track 10.0 -> 67.1 mm
- net ESP_RX: track 0.00 -> 53.8 mm, vias 0 -> 2
- net LED: track 0.00 -> 53.5 mm, vias 0 -> 2
- net Net-(K1-Pad3): track 10.0 -> 62.5 mm
- net TEMP_AMB: track 0.00 -> 44.4 mm, vias 0 -> 2
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
Commit message: pcb update
Parts:
- moved R1 4.50 mm to (232.5, 68.2)
- moved R12 4.50 mm to (232.5, 137.0)
- moved R16 4.50 mm to (232.5, 111.8)
- moved R5 4.50 mm to (232.5, 43.0)
- moved R11 3.00 mm to (224.0, 137.0)
- moved R15 3.00 mm to (224.0, 111.8)
- moved R2 3.00 mm to (224.0, 68.2)
- moved R6 3.00 mm to (224.0, 43.0)
- moved R10 1.50 mm to (215.5, 137.0)
- moved R14 1.50 mm to (215.5, 111.8)
- moved R3 1.50 mm to (215.5, 68.2)
- moved R7 1.50 mm to (215.5, 43.0)
Routing:
- net /VPOS: track 242.5 -> 231.9 mm
- net Net-(K15-Pad3): track 68.1 -> 64.4 mm
- net Net-(K11-Pad3): track 70.0 -> 67.0 mm
- net Net-(K12-Pad3): track 64.1 -> 61.3 mm
- net Net-(K14-Pad3): track 73.0 -> 70.3 mm
- net Net-(K16-Pad3): track 61.7 -> 59.4 mm
- net Net-(K6-Pad3): track 68.9 -> 66.6 mm
- net Net-(K1-Pad3): track 62.5 -> 60.6 mm
- net Net-(K5-Pad3): track 68.6 -> 66.7 mm
- net Net-(K10-Pad3): track 75.0 -> 73.5 mm
- net Net-(K2-Pad3): track 67.1 -> 65.9 mm
- net Net-(K7-Pad3): track 71.3 -> 70.7 mm
- net Net-(K3-Pad3): track 73.5 -> 72.8 mm
- net GND: vias 258 -> 166
- net +3.3V: vias 211 -> 121
Other:
- board text added: "+6V"
- board text added: "3.3V"
- board text added: "BOOT"
- board text added: "GND"
- board text added: "LOAD STEPPER V1.0"
- board text added: "NC"
- board text added: "RST"
- board text added: "RX"
- board text added: "TX"
- board text added: "VNEG"
- board text added: "VPOS"

Commit message: pcb update
Parts:
- moved U2 41.7 mm to (238.0, 72.5), turned to -90 degrees
- moved C5 41.5 mm to (238.8, 70.2), turned to 0 degrees
Routing:
- net +3.3V: track 28.2 -> 72.3 mm, vias 121 -> 147
- net TEMP_RES: track 126.6 -> 160.4 mm
- net GND: track 235.7 -> 217.7 mm, vias 166 -> 167
- net ESP_TX: track 58.8 -> 59.4 mm
- net ESP_RX: track 53.8 -> 54.4 mm
- added copper zone on F.Cu, net /VNEG
Other:
- board text added: "6.25Ω - 100Ω 4 Wmax Per"
