File: hw/relays.kicad_sch (KiCad schematic)
At the start: 128 parts, among them K1 G6K-2F-Y, K10 G6K-2F-Y, K11 G6K-2F-Y, K12 G6K-2F-Y, K13 G6K-2F-Y, K14 G6K-2F-Y, K15 G6K-2F-Y, K16 G6K-2F-Y, K2 G6K-2F-Y, K3 G6K-2F-Y, K4 G6K-2F-Y, K5 G6K-2F-Y, K6 G6K-2F-Y, K7 G6K-2F-Y, K8 G6K-2F-Y, K9 G6K-2F-Y, Q1 Si2302CDS, Q10 Si2302CDS, Q11 Si2302CDS, Q12 Si2302CDS, Q13 Si2302CDS, Q14 Si2302CDS, Q15 Si2302CDS, Q16 Si2302CDS, Q2 Si2302CDS, Q3 Si2302CDS, Q4 Si2302CDS, Q5 Si2302CDS, Q6 Si2302CDS, Q7 Si2302CDS, Q8 Si2302CDS, Q9 Si2302CDS

Commit message: sch & pcb update
Parts:
- added R61, R62, R63, R64, R65, R66, R67, R68, R69, R70, R71, R72, R73, R74, R75, R76: 10, Resistor_SMD:R_0603_1608Metric, symbol Device:R
- R15, R16, R19, R20, R27, R28, R31, R32, R39, R40, R43, R44, R51, R52, R55, R56: jlc_part C118155 -> C21190; mfr_part ERJ3EKF1001V -> 0603WAF1001T5E
Connections:
- net P00: now also R61.2; no longer C21.1, Q1.1 (G), R13.2
- net P01: now also R65.2; no longer C25.1, Q5.1 (G), R25.2
- net P02: now also R69.2; no longer C29.1, Q9.1 (G), R37.2
- net P03: now also R73.2; no longer C33.1, Q13.1 (G), R49.2
- net P04: now also R62.2; no longer C22.1, Q2.1 (G), R14.2
- net P05: now also R66.2; no longer C26.1, Q6.1 (G), R26.2
- net P06: now also R70.2; no longer C30.1, Q10.1 (G), R38.2
- net P07: now also R74.2; no longer C34.1, Q14.1 (G), R50.2
- net P10: now also R63.2; no longer C23.1, Q3.1 (G), R17.2
- net P11: now also R67.2; no longer C27.1, Q7.1 (G), R29.2
- net P12: now also R71.2; no longer C31.1, Q11.1 (G), R41.2
- net P13: now also R75.2; no longer C35.1, Q15.1 (G), R53.2
- net P14: now also R64.2; no longer C24.1, Q4.1 (G), R18.2
- net P15: now also R68.2; no longer C28.1, Q8.1 (G), R30.2
- net P16: now also R72.2; no longer C32.1, Q12.1 (G), R42.2
- net P17: now also R76.2; no longer C36.1, Q16.1 (G), R54.2
- new net: C27.1, Q7.1 (G), R29.2, R67.1
- new net: C36.1, Q16.1 (G), R54.2, R76.1
- new net: C33.1, Q13.1 (G), R49.2, R73.1
- new net: C31.1, Q11.1 (G), R41.2, R71.1
- new net: C28.1, Q8.1 (G), R30.2, R68.1
- new net: C30.1, Q10.1 (G), R38.2, R70.1
- new net: C25.1, Q5.1 (G), R25.2, R65.1
- new net: C22.1, Q2.1 (G), R14.2, R62.1
- new net: C29.1, Q9.1 (G), R37.2, R69.1
- new net: C35.1, Q15.1 (G), R53.2, R75.1
- new net: C23.1, Q3.1 (G), R17.2, R63.1
- new net: C32.1, Q12.1 (G), R42.2, R72.1
- new net: C24.1, Q4.1 (G), R18.2, R64.1
- new net: C21.1, Q1.1 (G), R13.2, R61.1
- new net: C34.1, Q14.1 (G), R50.2, R74.1
- new net: C26.1, Q6.1 (G), R26.2, R66.1
Other:
- moved on the sheet: C23, C24, C27, C28, C31, C32, C35, C36, D10, D11, D12, D13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

Commit message: pcb update
Parts:
- renumbered C25 to C22, C29 to C23, C33 to C24, C22 to C25, C30 to C27, C34 to C28, C23 to C29, C27 to C30, C35 to C32, C24 to C33, C28 to C34, C32 to C35, D30 to D10, D8 to D11, D16 to D12, D24 to D13, D32 to D14, D7 to D15, D15 to D16, D23 to D17, D31 to D18, D9 to D19, D17 to D20, D25 to D21, D33 to D22, D10 to D23, D18 to D24, D26 to D25, D34 to D26, D12 to D27, D20 to D28, D28 to D29, D36 to D30, D11 to D31, D19 to D32, D27 to D33, D35 to D34, D13 to D35, D21 to D36, D29 to D37, D37 to D38, D6 to D7, D14 to D8, D22 to D9, K7 to K10, K15 to K12, K4 to K13, K8 to K14, K12 to K15, K5 to K2, K9 to K3, K13 to K4, K2 to K5, K10 to K7, K14 to K8, K3 to K9, Q7 to Q10, Q15 to Q12, Q4 to Q13, Q8 to Q14, Q12 to Q15, Q5 to Q2, Q9 to Q3, Q13 to Q4, Q2 to Q5, Q10 to Q7, Q14 to Q8, Q3 to Q9, R21 to R1, R35 to R10, R47 to R11, R59 to R12, R24 to R13, R36 to R14, R48 to R15, R60 to R16, R33 to R2, R45 to R3, R15 to R31, R27 to R32, R39 to R33, R51 to R34, R61 to R35, R65 to R36, R69 to R37, R73 to R38, R13 to R39, R57 to R4, R25 to R40, R37 to R41, R49 to R42, R16 to R43, R28 to R44, R40 to R45, R52 to R46, R62 to R47, R66 to R48, R70 to R49, R22 to R5, R74 to R50, R14 to R51, R26 to R52, R38 to R53, R50 to R54, R19 to R55, R31 to R56, R43 to R57, R55 to R58, R63 to R59, R34 to R6, R67 to R60, R71 to R61, R75 to R62, R17 to R63, R29 to R64, R41 to R65, R53 to R66, R20 to R67, R32 to R68, R44 to R69, R46 to R7, R56 to R70, R64 to R71, R68 to R72, R72 to R73, R76 to R74, R18 to R75, R30 to R76, R42 to R77, R54 to R78, R58 to R8, R23 to R9

Commit message: pcb update
Parts:
- D10, D15, D16, D17, D18, D23, D24, D25, D26, D31, D32, D33, D34, D7, D8, D9: jlc_part C2986060 -> C2286; mfr_part 19-217/R6C-AL1M2VY/6T -> KT-0603R
- D11, D12, D13, D14, D19, D20, D21, D22, D27, D28, D29, D30, D35, D36, D37, D38: footprint Diode_SMD:D_SOD-323_HandSoldering -> Diode_SMD:D_SOD-323
- K1, K10, K11, K12, K13, K14, K15, K16, K2, K3, K4, K5, K6, K7, K8, K9: jlc_part (none) -> C2153097; mfr_part (none) -> G6K-2F-Y-TR DC3
- R1, R10, R11, R12, R13, R14, R15, R16, R2, R3, R4, R5, R6, R7, R8, R9: now not fitted; now left out of the parts list

Commit message: pcb completed
Parts:
- K1, K10, K11, K12, K13, K14, K15, K16, K2, K3, K4, K5, K6, K7, K8, K9: now not fitted; now left out of the parts list
Changed lines of the file:
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@@
 		(unit 1)
 		(exclude_from_sim no)
-		(in_bom yes)
+		(in_bom no)
 		(on_board yes)
-		(dnp no)
+		(dnp yes)
 		(property "Reference" "K3"
 			(at 280.67 36.8299 0)
@@
 		(unit 1)
 		(exclude_from_sim no)
-		(in_bom yes)
+		(in_bom no)
 		(on_board yes)
-		(dnp no)
+		(dnp yes)
 		(property "Reference" "K6"
 			(at 191.77 100.3299 0)
@@
 		(unit 1)
 		(exclude_from_sim no)
-		(in_bom yes)
+		(in_bom no)
 		(on_board yes)
-		(dnp no)
+		(dnp yes)
 		(property "Reference" "K11"
 			(at 280.67 163.8299 0)
@@
 		(unit 1)
 		(exclude_from_sim no)
-		(in_bom yes)
+		(in_bom no)
 		(on_board yes)
-		(dnp no)
+		(dnp yes)
 		(property "Reference" "K14"
 			(at 191.77 227.3299 0)
@@
 		(unit 1)
 		(exclude_from_sim no)
-		(in_bom yes)
+		(in_bom no)
 		(on_board yes)
-		(dnp no)
+		(dnp yes)
 		(property "Reference" "K10"
 			(at 191.77 163.8299 0)
@@
 		(unit 1)
 		(exclude_from_sim no)
-		(in_bom yes)
+		(in_bom no)
 		(on_board yes)
-		(dnp no)
+		(dnp yes)
 		(property "Reference" "K4"
 			(at 369.57 36.8299 0)
@@
 		(unit 1)
 		(exclude_from_sim no)
-		(in_bom yes)
+		(in_bom no)
 		(on_board yes)
-		(dnp no)
+		(dnp yes)
 		(property "Reference" "K15"
 			(at 280.67 227.3299 0)
@@
 		(unit 1)
 		(exclude_from_sim no)
-		(in_bom yes)
+		(in_bom no)
 		(on_board yes)
-		(dnp no)
+		(dnp yes)
 		(property "Reference" "K5"
 			(at 102.87 100.3299 0)
@@
 		(unit 1)
 		(exclude_from_sim no)
-		(in_bom yes)
+		(in_bom no)
 		(on_board yes)
-		(dnp no)
+		(dnp yes)
 		(property "Reference" "K12"
 			(at 369.57 163.8299 0)
@@
 		(unit 1)
 		(exclude_from_sim no)
-		(in_bom yes)
+		(in_bom no)
 		(on_board yes)
-		(dnp no)
+		(dnp yes)
 		(property "Reference" "K16"
 			(at 369.57 227.3299 0)
@@
 		(unit 1)
 		(exclude_from_sim no)
-		(in_bom yes)
+		(in_bom no)
 		(on_board yes)
-		(dnp no)
+		(dnp yes)
 		(property "Reference" "K1"
 			(at 102.87 36.8299 0)
@@
 		(unit 1)
 		(exclude_from_sim no)
-		(in_bom yes)
+		(in_bom no)
 		(on_board yes)
-		(dnp no)
+		(dnp yes)
 		(property "Reference" "K8"
 			(at 369.57 100.3299 0)
@@
 		(unit 1)
 		(exclude_from_sim no)
-		(in_bom yes)
+		(in_bom no)
 		(on_board yes)
-		(dnp no)
+		(dnp yes)
 		(property "Reference" "K2"
 			(at 191.77 36.8299 0)
@@
 		(unit 1)
 		(exclude_from_sim no)
-		(in_bom yes)
+		(in_bom no)
 		(on_board yes)
-		(dnp no)
+		(dnp yes)
 		(property "Reference" "K9"
 			(at 102.87 163.8299 0)
@@
 		(unit 1)
 		(exclude_from_sim no)
-		(in_bom yes)
+		(in_bom no)
 		(on_board yes)
-		(dnp no)
+		(dnp yes)
 		(property "Reference" "K13"
 			(at 102.87 227.3299 0)
@@
 		(unit 1)
 		(exclude_from_sim no)
-		(in_bom yes)
+		(in_bom no)
 		(on_board yes)
-		(dnp no)
+		(dnp yes)
 		(property "Reference" "K7"
 			(at 280.67 100.3299 0)
